Commit message: 1.1

File: src/dual_arm_description/urdf/arm.xacro (robot description, xacro)
@@ -4,6 +4,6 @@
   <xacro:macro name="arm" params="prefix side">
     <joint name="${prefix}_mount_joint" type="fixed">
-      <parent link="base_link"/><child link="${prefix}_mount_link"/>
-      <origin xyz="0 ${side*mount_spacing/2} ${mount_height}"/>
+      <parent link="crossbar_link"/><child link="${prefix}_mount_link"/>
+      <origin xyz="0 ${side*mount_spacing/2} ${crossbar_height/2+0.038}"/>
     </joint>
     <link name="${prefix}_mount_link">
@@ -13,6 +13,5 @@
     </link>
     <xacro:hinge name="${prefix}_shoulder_pitch_joint" parent="${prefix}_mount_link"
-                 child="${prefix}_shoulder_link" xyz="0 ${side*0.022} 0" axis="0 -1 0"
-                 lower="${-pi/2}" upper="${pi/2}"/>
+                 child="${prefix}_shoulder_link" xyz="0 ${side*0.022} 0" axis="0 -1 0"/>
     <link name="${prefix}_shoulder_link">
       <!-- The second motor's long case points inward to the first motor.
@@ -28,6 +27,5 @@
                              scale="1 ${(d['shoulder_outboard']-0.038)/0.002} 1"/>
     <xacro:hinge name="${prefix}_shoulder_roll_joint" parent="${prefix}_shoulder_link"
-                 child="${prefix}_upper_arm_link" xyz="0 ${side*d['shoulder_outboard']} 0" axis="${side} 0 0"
-                 lower="${-pi/3}" upper="${pi/2}"/>
+                 child="${prefix}_upper_arm_link" xyz="0 ${side*d['shoulder_outboard']} 0" axis="${side} 0 0"/>
     <link name="${prefix}_upper_arm_link">
       <xacro:mesh_visual mesh="shoulder_fork" material="frame_grey"/>
@@ -48,6 +46,5 @@
     <!-- Elbow casing is downstream; upper fork holds its output horn. -->
     <xacro:hinge name="${prefix}_elbow_pitch_joint" parent="${prefix}_upper_arm_link"
-                 child="${prefix}_forearm_link" xyz="0 0 ${-d['upper_arm_length']}" axis="0 -1 0"
-                 lower="${-pi/2}" upper="${pi/2}"/>
+                 child="${prefix}_forearm_link" xyz="0 0 ${-d['upper_arm_length']}" axis="0 -1 0"/>
     <link name="${prefix}_forearm_link">
       <xacro:servo rpy="0 0 ${pi/2}"/>
@@ -66,6 +63,5 @@
                              scale="1 1 ${(d['wrist_drop']-0.033)/0.040}"/>
     <xacro:hinge name="${prefix}_wrist_roll_joint" parent="${prefix}_forearm_link"
-                 child="${prefix}_palm_link" xyz="${wrist_axis_x} 0 ${-d['wrist_drop']}" axis="0 0 -1"
-                 lower="${-pi/2}" upper="${pi/2}"/>
+                 child="${prefix}_palm_link" xyz="${wrist_axis_x} 0 ${-d['wrist_drop']}" axis="0 0 -1"/>
     <link name="${prefix}_palm_link">
       <!-- The hand has its own centreline; do not centre it on the wrist housing. -->
@@ -93,5 +89,5 @@
     <xacro:hinge name="${prefix}_${role}_finger_joint" parent="${prefix}_palm_link"
                  child="${prefix}_${role}_finger_link" xyz="${mount_x} ${direction*d['finger_spacing']/2} ${-d['palm_drop']}"
-                 axis="${direction} 0 0" lower="0" upper="${pi/3}"/>
+                 axis="${direction} 0 0"/>
     <link name="${prefix}_${role}_finger_link">
       <xacro:mesh_visual mesh="${mesh}" material="frame_grey" rpy="0 0 ${0 if direction == 1 else pi}"/>

File: src/dual_arm_description/urdf/components.xacro (robot description, xacro)
@@ -39,9 +39,11 @@
     <xacro:mesh_visual mesh="ax12a_lettering" material="servo_black" xyz="${xyz}" rpy="${rpy}"/>
   </xacro:macro>
-  <xacro:macro name="hinge" params="name parent child xyz axis lower upper">
+  <xacro:macro name="hinge" params="name parent child xyz axis">
+    <xacro:property name="limits" value="${joint_limits[name]}"/>
     <joint name="${name}" type="revolute">
       <parent link="${parent}"/><child link="${child}"/>
       <origin xyz="${xyz}"/><axis xyz="${axis}"/>
-      <limit lower="${lower}" upper="${upper}" effort="${d['arm_effort']}" velocity="${d['arm_velocity']}"/>
+      <limit lower="${limits['min_position_deg']*pi/180}" upper="${limits['max_position_deg']*pi/180}"
+             effort="${limits['max_effort_nm']}" velocity="${limits['max_velocity_deg_s']*pi/180}"/>
       <dynamics damping="0.02" friction="0.01"/>
     </joint>

File: src/dual_arm_description/urdf/dual_arm.urdf (robot description, URDF)
Before this commit: robot bioloid_dual_arm, 23 links, 22 joints
Links:
- added link crossbar_link, mass 0.2; collision box size=0.04 0.158 0.02; visual mesh filename=package://dual_arm_description/meshes/aluminum_crossbar.stl scale=1 1 1
Joints:
- added joint crossbar_mount_joint: type fixed, parent base_link, child crossbar_link, origin xyz=0 0 0.342
- joint left_elbow_pitch_joint: limit lower=-1.5707963267948966 upper=1.5707963267948966 effort=0.3 velocity=1.0 -> lower=0.0 upper=1.5707963267948966 effort=0.3 velocity=0.3490658503988659
- joint left_inner_finger_joint: limit lower=0 upper=1.0471975511965976 effort=0.3 velocity=1.0 -> lower=0.0 upper=0.5235987755982988 effort=0.3 velocity=0.5235987755982988
- joint left_mount_joint: origin xyz=0 0.12 0.39 -> xyz=0 0.059 0.048; parent base_link -> crossbar_link
- joint left_outer_finger_joint: limit lower=0 upper=1.0471975511965976 effort=0.3 velocity=1.0 -> lower=0.0 upper=0.5235987755982988 effort=0.3 velocity=0.5235987755982988
- joint left_shoulder_pitch_joint: limit lower=-1.5707963267948966 upper=1.5707963267948966 effort=0.3 velocity=1.0 -> lower=-0.5235987755982988 upper=1.0471975511965976 effort=0.3 velocity=0.3490658503988659
- joint left_shoulder_roll_joint: limit lower=-1.0471975511965976 upper=1.5707963267948966 effort=0.3 velocity=1.0 -> lower=0.0 upper=0.7853981633974483 effort=0.3 velocity=0.3490658503988659
- joint left_wrist_roll_joint: limit lower=-1.5707963267948966 upper=1.5707963267948966 effort=0.3 velocity=1.0 -> lower=-1.1780972450961724 upper=1.1780972450961724 effort=0.3 velocity=0.3490658503988659
- joint right_elbow_pitch_joint: limit lower=-1.5707963267948966 upper=1.5707963267948966 effort=0.3 velocity=1.0 -> lower=0.0 upper=1.5707963267948966 effort=0.3 velocity=0.3490658503988659
- joint right_inner_finger_joint: limit lower=0 upper=1.0471975511965976 effort=0.3 velocity=1.0 -> lower=0.0 upper=0.5235987755982988 effort=0.3 velocity=0.5235987755982988
- joint right_mount_joint: origin xyz=0 -0.12 0.39 -> xyz=0 -0.059 0.048; parent base_link -> crossbar_link
- joint right_outer_finger_joint: limit lower=0 upper=1.0471975511965976 effort=0.3 velocity=1.0 -> lower=0.0 upper=0.5235987755982988 effort=0.3 velocity=0.5235987755982988
- joint right_shoulder_pitch_joint: limit lower=-1.5707963267948966 upper=1.5707963267948966 effort=0.3 velocity=1.0 -> lower=-0.5235987755982988 upper=1.0471975511965976 effort=0.3 velocity=0.3490658503988659
- joint right_shoulder_roll_joint: limit lower=-1.0471975511965976 upper=1.5707963267948966 effort=0.3 velocity=1.0 -> lower=0.0 upper=0.7853981633974483 effort=0.3 velocity=0.3490658503988659
- joint right_wrist_roll_joint: limit lower=-1.5707963267948966 upper=1.5707963267948966 effort=0.3 velocity=1.0 -> lower=-1.1780972450961724 upper=1.1780972450961724 effort=0.3 velocity=0.3490658503988659

File: src/dual_arm_description/urdf/dual_arm.urdf.xacro (robot description, xacro)
@@ -3,5 +3,12 @@
   <xacro:arg name="dimensions_file" default="$(find dual_arm_description)/config/dimensions.yaml"/>
   <xacro:property name="d" value="${xacro.load_yaml('$(arg dimensions_file)')}"/>
-  <xacro:arg name="mount_spacing" default="${d['mount_spacing']}"/>
+  <xacro:property name="joint_limits" value="${xacro.load_yaml('$(find dual_arm_description)/config/joint_limits.yaml')['joint_limits']}"/>
+  <xacro:property name="parts" value="${xacro.load_yaml('$(find dual_arm_description)/config/parts.yaml')}"/>
+  <xacro:property name="crossbar" value="${parts['aluminum_crossbar']}"/>
+  <!-- User dimensions are mm; URDF geometry is expressed in metres. -->
+  <xacro:property name="crossbar_length" value="${crossbar['length_mm']/1000.0}"/>
+  <xacro:property name="crossbar_depth" value="${crossbar['depth_mm']/1000.0}"/>
+  <xacro:property name="crossbar_height" value="${crossbar['height_mm']/1000.0}"/>
+  <xacro:arg name="mount_spacing" default="${d.get('mount_spacing', crossbar_length-0.040)}"/>
   <xacro:arg name="mount_height" default="${d['mount_height']}"/>
   <xacro:property name="mount_spacing" value="$(arg mount_spacing)"/>
@@ -11,6 +18,18 @@
   <xacro:include filename="components.xacro"/>
   <xacro:include filename="arm.xacro"/>
-  <!-- Virtual assembly datum only: no fabricated torso/stand geometry. -->
+  <!-- Keep the floor datum massless; the physical crossbar supports both arms. -->
   <link name="base_link"/>
+  <joint name="crossbar_mount_joint" type="fixed">
+    <parent link="base_link"/><child link="crossbar_link"/>
+    <!-- Shoulder case bottom is 38 mm below its shaft in the current mesh. -->
+    <origin xyz="0 0 ${mount_height-0.038-crossbar_height/2}"/>
+  </joint>
+  <link name="crossbar_link">
+    <xacro:mesh_visual mesh="aluminum_crossbar" material="servo_black"/>
+    <xacro:box_collision size="${crossbar_depth} ${crossbar_length} ${crossbar_height}"/>
+    <!-- Wall thickness is unspecified: uniform outer-box inertia approximation. -->
+    <xacro:box_inertia mass="${crossbar['mass_kg']}" x="${crossbar_depth}"
+                       y="${crossbar_length}" z="${crossbar_height}"/>
+  </link>
   <xacro:arm prefix="left" side="1"/>
   <xacro:arm prefix="right" side="-1"/>
