Commit message: 2.0

File: src/dual_arm_description/urdf/dual_arm.urdf (robot description, URDF)
Before this commit: robot bioloid_dual_arm, 24 links, 23 joints
Joints:
- joint left_shoulder_pitch_joint: limit lower=-0.5235987755982988 upper=1.0471975511965976 effort=0.3 velocity=0.3490658503988659 -> lower=-0.5235987755982988 upper=1.5707963267948966 effort=0.3 velocity=0.3490658503988659
- joint left_shoulder_roll_joint: limit lower=0.0 upper=0.7853981633974483 effort=0.3 velocity=0.3490658503988659 -> lower=0.0 upper=1.5707963267948966 effort=0.3 velocity=0.3490658503988659
- joint right_shoulder_pitch_joint: limit lower=-0.5235987755982988 upper=1.0471975511965976 effort=0.3 velocity=0.3490658503988659 -> lower=-0.5235987755982988 upper=1.5707963267948966 effort=0.3 velocity=0.3490658503988659
- joint right_shoulder_roll_joint: limit lower=0.0 upper=0.7853981633974483 effort=0.3 velocity=0.3490658503988659 -> lower=0.0 upper=1.5707963267948966 effort=0.3 velocity=0.3490658503988659
